File: kicad/papertape_panel.kicad_pcb (KiCad board)
At the start: 2 copper layers, 210 x 88.9 mm, 184 parts, among them T1 BPW17N, T2 BPW17N, T3 BPW17N, T4 BPW17N, T5 BPW17N, T6 BPW17N, T7 BPW17N, T8 BPW17N, T9 BPW17N, U1 PRO_MICRO

Commit message: Add panel silkscreen notes for feed-track blind-hole drilling.
Mark the correct drill side and point builders to README drilling instructions.

Co-authored-by: Cursor <cursoragent@cursor.com>
Other:
- board text added: "DO NOT DRILL FROM THIS SIDE!"
- board text added: "IMPORTANT INFO IN README!"
Changed lines of the file:
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@@
 		(layer "User.5")
+	)
+	(gr_text "IMPORTANT INFO IN README!"
+		(at 87.4 57.4 0)
+		(layer "F.SilkS")
+		(effects
+			(font
+				(size 1 1)
+				(thickness 0.1)
+			)
+			(justify left bottom)
+		)
 	)
 	(gr_text "Blind hole 1.8mm\nfor phototransistor"
@@
 		)
 	)
+	(gr_text "IMPORTANT INFO IN README!"
+		(at 109 103 0)
+		(layer "B.SilkS")
+		(effects
+			(font
+				(size 1 1)
+				(thickness 0.1)
+			)
+			(justify left bottom mirror)
+		)
+	)
+	(gr_text "DO NOT DRILL FROM  THIS SIDE!"
+		(at 111 105 0)
+		(layer "B.SilkS")
+		(effects
+			(font
+				(size 1 1)
+				(thickness 0.1)
+			)
+			(justify left bottom mirror)
+		)
+	)
